File: BeagleBone_Blue.sch (EAGLE design)
At the start: 282 parts, among them J1 68000-406HLF, P2 CTIJTAG, P3 87520-0010BLF, U10 TPD4S012, U12 MT41K256M16HA, U13 MTFC4GLDEA, U15 SN74LVC2G241DCU, U16 SN74LVC1G07DCK, U3 SN74LVC1G06DCK, U4 TL5209, U5 AM3358_BZCZ_324, U6 SN74LVC1G74_DCT_8, U7 24LC_32AT-I/OT, U8 TPS2051BD, U9 TPD4S012, Y1 CM200C-32.768KAZF-UT, Y2 445C33D24M00000, Y4 ASDMB-24.576MHZ-LC-T

Commit message: remove and put robotics cape components back to try to fix ERC errors. failed. :(
Parts:
- added 5VREG: AP1509SOIC-8-TIGHT, Strawson_Eagle_Lib:AP1509SOIC-8-TIGHT
- added 6V_REG: AOZ1284, Strawson_Eagle_Lib:AOZ1284
- added ADC, GPS, SPI1.1, SPI1.2: JST_SH_6, Strawson_Eagle_Lib:JST_SH_6
- added BAL: BQ29209, Strawson_Eagle_Lib:BQ29209
- added BMP: BMP180, SparkFun-Sensors:BMP180
- added C131, C138, C139, C140, C141, C142, C143, C145, C146, C148, C149, C23, C24, C5: 0.1uF, Strawson_Eagle_Lib:CAP0402-CAP
- added C132: 100uF 16V, adafruit:CPOL-USD
- added C133, C134, C135, C136, C137, C144, C147, C150, C151: 10uF 25V, SparkFun-Capacitors:CAP0805
- added C25, C6: 1uF, Strawson_Eagle_Lib:CAP0402-CAP
- added CHG, GRN: GRN, SparkFun-LED:LED0603
- added CHGIC: MP2615, Strawson_Eagle_Lib:MP2615
- added D10, RED: RED, SparkFun-LED:LED0603
- added D11, D12, D9: GREEN, SparkFun-LED:LED0603
- added D13: (no value), Strawson_Eagle_Lib:DIODEDO214AA
- added D6, D7, D8: (no value), adafruit:DIODESOD-123
- added DSM2: JST_ZH_3, Strawson_Eagle_Lib:JST_ZH_3
- added E1, E2, E3, E4, I2C1, PWR, UART1, UART5: JST_SH_4, Strawson_Eagle_Lib:JST_SH_4
- added H1, H2: TB6621FNG, SparkFun:TB6621FNG
- added IMU: MPU-9250, Strawson_Eagle_Lib:MPU-9250
- added JACK: 5.5x2.1mm, con-jack:DCJ0303
- added L4, L5: 6.8uH, SparkFun-Passives:INDUCTORBOURNS_SRN6045
- added L6: 3.6, Strawson_Eagle_Lib:INDUCTOR
- added LIPO: (no value), Strawson_Eagle_Lib:JST_XH_3-PIN
- added M1, M2, M3, M4: JST_ZH_2, Strawson_Eagle_Lib:JST_ZH_2
- added MODE, PAUSE, POWER, RESET: SWITCH-MOMENTARY-2-SMD-1101NE, SparkFun-Electromechanical:SWITCH-MOMENTARY-2-SMD-1101NE
- added PROT: S-8261, Strawson_Eagle_Lib:S-8261
- added Q3: MOSFET-N, Strawson_Eagle_Lib:MOSFET-NCHANNEL
- added R113, R114, R115, R116, R117, R118, R119, R120, R121, R134, R135, R136, R137, R138, R139, R14, R140, R141, R142, R15, R16, R27, R34: 4.7k, Strawson_Eagle_Lib:RESISTOR0402-RES
- added R122, R123, R125: 160, Strawson_Eagle_Lib:RESISTOR0402-RES
- added R124, R31, R32, R41, R42, R43, R44: 261, Strawson_Eagle_Lib:RESISTOR0402-RES
- added R126, R127, R133, R35, R36, R37, R38, R39, R40: 1K, Strawson_Eagle_Lib:RESISTOR0402-RES
- added R128, R2: 1k, Strawson_Eagle_Lib:RESISTOR0402-RES
- added R129, R33, R51: 47k, Strawson_Eagle_Lib:RESISTOR0402-RES
- added R13, R131, R143, R9: 10k, Strawson_Eagle_Lib:RESISTOR0402-RES
- added R130: 100k, Strawson_Eagle_Lib:RESISTOR0402-RES
- added R132: 65k, Strawson_Eagle_Lib:RESISTOR0402-RES
- added R6: 0.1, SparkFun-Resistors:RESISTOR0603
- added U$7: SERVO_HEADERS_8X, Strawson_Eagle_Lib:SERVO_HEADERS_8X
Connections:
- new net 3.3V: BMP.VDD, BMP.VDDIO, C137.1, C138.1, C149.2, C24.1, C5.2, DSM2.1, E1.2, E2.2, E3.2, E4.2, H1.VCC, H2.VCC, I2C1.2, IMU.NCS, IMU.RESV, IMU.VDD, IMU.VDDIO, PWR.3, R126.2, R127.2, R14.1, R15.2, R16.2, R27.1, R35.2, R36.2, R37.2, R38.2, R39.2, R40.2, SPI1.1.2, SPI1.2.2, UART1.2, UART5.2
- new net 5.0V: 5VREG.FB, C134.1, GPS.5, L5.2, PWR.4
- new net BATT_MID: LIPO.2, R122.1, R124.1, R128.1
- new net BATT_MINUS: BAL.CB_EN, BAL.GND, C140.1, C141.2, C142.2, C143.1, LIPO.3, PROT.VM, PROT.VSS, Q3.S
- new net CHG_EN: CHGIC.EN, R142.2, R143.1
- new net CO: BAL.OUT, R142.1
- new net DO: PROT.DO, Q3.G
- new net L3: D12.C, R44.1
- new net L4: D11.C, R43.1
- new net MOT1A: H1.A01@1, H1.A01@2, M1.2
- new net MOT1B: H1.A02@5, H1.A02@6, M1.1
- new net MOT2A: H1.B01@11, H1.B01@12, M2.1
- new net MOT2B: H1.B02@7, H1.B02@8, M2.2
- new net MOT3A: H2.A01@1, H2.A01@2, M3.1
- new net MOT3B: H2.A02@5, H2.A02@6, M3.2
- new net MOT4A: H2.B01@11, H2.B01@12, M4.2
- new net MOT4B: H2.B02@7, H2.B02@8, M4.1
- new net N$10: BAL.VC1, C139.1, C140.2, R124.2
- new net N$11: BAL.VC2, C139.2, R123.2
- new net N$12: C143.2, PROT.VDD, R128.2
- new net N$13: 6V_REG.SS, C145.2
- new net N$14: C23.1, IMU.REGOUT
- new net N$15: C131.1, CHGIC.BST
- new net N$16: 5VREG.OUT, D6.C, L5.1
- new net N$18: CHGIC.CHGOK, R2.1
- new net N$20: CHGIC.NTC, R13.2, R9.1
- new net N$24: BAL.CD, C141.1
- new net N$25: R115.2, U$7.2
- new net N$29: BAL.VDD, C142.1, R125.2
- new net N$30: R116.2, U$7.3
- new net N$38: R117.2, U$7.4
- new net N$4: CHG.C, R2.2
- new net N$48: D9.C, R41.1
- new net N$49: D10.C, R42.1
- new net N$5: GRN.C, R32.1
- new net N$50: BAL.VC1_CB, R122.2
- new net N$51: R118.2, U$7.5
- new net N$52: R119.2, U$7.6
- new net N$53: 6V_REG.BS, C146.1
- new net N$54: R120.2, U$7.7
- new net N$55: C131.2, CHGIC.SW, L4.1
- new net N$56: R121.2, U$7.8
- new net N$6: R31.1, RED.C
- new net N$60: 6V_REG.LX, C146.2, D13.C, L6.1
- new net N$61: 6V_REG.FSW, R130.2
- new net N$62: C147.2, L6.2, R132.2, U$7.PWR
- new net N$63: 6V_REG.COMP, R129.2
- new net N$65: 6V_REG.FB, R131.2, R132.1
- new net N$66: C148.2, R129.1
- new net N$67: CHGIC.CSP, L4.2, R6.2
- new net N$69: C6.2, CHGIC.TMR
- new net N$7: R114.2, U$7.1
- new net N$79: 5VREG.VIN, C133.1, D7.C, D8.C
- new net PWR: POWER.2
- new net RESET: RESET.2
- new net SPI1_SCK: SPI1.1.5, SPI1.2.5
- new net SPI1_SS1: SPI1.1.6
- new net VCC_CHG: C25.2, CHGIC.SEL, CHGIC.VCC, R9.2
- new net VDD_ADC: ADC.2
- new net V_BATT: 6V_REG.VIN, C132.+, C144.2, C150.1, C151.1, CHGIC.BATT, D7.A, H1.VM1, H1.VM2, H1.VM3, H2.VM1, H2.VM2, H2.VM3, LIPO.1, R123.1, R125.1, R33.1, R6.1
- new net V_DIV_BAT: R33.2, R34.1
- new net V_DIV_DC: R113.1, R51.2
- net AIN0: now also ADC.3
- net AIN1: now also ADC.4
- net AIN2: now also ADC.5
- net AIN3: now also ADC.6
- net GND: now also 5VREG.GND, 5VREG.GND1, 5VREG.GND2, 5VREG.GND3, 5VREG.SD, 6V_REG.GND, ADC.1, BMP.GND, C132.-, C133.2, C134.2, C135.2, C136.2, C137.2, C138.2, C144.1, C145.1, C147.1, C148.1, C149.1, C150.2, C151.2, C23.2, C24.2, C25.1, C5.1, C6.1, CHGIC.AGND, CHGIC.PGND, D13.A, D6.A, DSM2.2, E1.1, E2.1, E3.1, E4.1, GPS.2, GPS.6, H1.GND, H1.PGND1@3, H1.PGND1@4, H1.PGND2@10, H1.PGND2@9, H2.GND, H2.PGND1@3, H2.PGND1@4, H2.PGND2@10, H2.PGND2@9, I2C1.1, IMU.AD0/SDO, IMU.GND, IMU.PAD, IMU.RESV@2, JACK.2, JACK.3, MODE.1, PAUSE.1, POWER.1, PWR.1, PWR.2, Q3.D, R113.2, R13.1, R130.1, R131.1, R133.1, R134.2, R135.2, R136.2, R137.2, R138.1, R139.1, R140.1, R141.1, R143.2, R31.2, R32.2, R34.2, R41.2, R42.2, R43.2, R44.2, RESET.1, SPI1.1.1, SPI1.2.1, U$7.GND, UART1.1, UART5.1
- net I2C1_SCL: now also I2C1.3, R16.1
- net I2C1_SDA: now also I2C1.4, R27.2
- net I2C2_SCL: now also BMP.SCL, IMU.SCL/SCLK, R15.1
- net I2C2_SDA: now also BMP.SDA, IMU.SDA/SDI, R14.2
- net IMU_INT: now also IMU.INT
- net LED_1: now also D10.A
- net LED_2: now also D9.A
- net LED_3: now also D12.A
- net LED_4: now also D11.A
- net LED_GRN: now also GRN.A
- net LED_RED: now also RED.A
- net MDIR_1A: now also H1.AIN1
- net MDIR_1B: now also H1.AIN2
- net MDIR_2A: now also H1.BIN1
- net MDIR_2B: now also H1.BIN2
- net MDIR_3A: now also H2.AIN1
- net MDIR_3B: now also H2.AIN2
- net MDIR_4A: now also H2.BIN1
- net MDIR_4B: now also H2.BIN2
- net MODE_BTN: now also MODE.2
- net MOT_STBY: now also H1.STBY, H2.STBY
- net PAUSE_BTN: now also PAUSE.2
- net PWM_1A: now also H1.PWMA
- net PWM_1B: now also H1.PWMB
- net PWM_2A: now also H2.PWMA
- net PWM_2B: now also H2.PWMB
- net QEP_0A: now also E1.3, R40.1
- net QEP_0B: now also E1.4, R39.1
- net QEP_1A: now also E2.3, R38.1
- net QEP_1B: now also E2.4, R37.1
- net QEP_2A: now also E3.3, R36.1
- net QEP_2B: now also E3.4, R35.1
- net QEP_4A: now also E4.3, R127.1
- net QEP_4B: now also E4.4, R126.1
- net SERVO_EN: now also 6V_REG.EN, R133.2
- net SPI1_MISO: now also SPI1.1.4, SPI1.2.4
- net SPI1_MOSI: now also SPI1.1.3, SPI1.2.3
- net SPI1_SS2: now also SPI1.2.6
- net SVO1: now also R114.1, R134.1
- net SVO2: now also R115.1, R135.1
- net SVO3: now also R116.1, R136.1
- net SVO4: now also R117.1, R137.1
- net SVO5: now also R118.1, R138.2
- net SVO6: now also R119.1, R139.2
- net SVO7: now also R120.1, R140.2
- net SVO8: now also R121.1, R141.2
- net UART1_RX: now also UART1.3
- net UART1_TX: now also UART1.4
- net UART2_RX: now also GPS.3
- net UART2_TX: now also GPS.4
- net UART4_RX: now also DSM2.3
- net UART5_RX: now also UART5.3
- net UART5_TX: now also UART5.4
- net VCC: now also C135.1, C136.1, CHG.A, CHGIC.VIN, D8.A, JACK.1, R51.1
Other:
- note added: "0.1 Ohm resistor for 1A charge"
- note added: "2A 5V Regulator"
- note added: "2S LiPo Charger"
- note added: "2S Lithium Balancer and Protection"
- note added: "ADC Dividers"
- note added: "Barometer"
- note added: "Barrel Connector Center Positive 5.5x2.1mm"
- note added: "Battery Connector"
- note added: "Battery Indicator LEDs"
- note added: "Buttons and LEDs"
- note added: "CELL pin left open: 2S SEL pin pulled HIGH: charge to 4.1V per cell"
- note added: "For EM-506 GPS Style Connector"
- note added: "I2C Pullups"
- note added: "IMU 9-Axis"
- note added: "JST XH"
- note added: "JST-SH"
- note added: "JST-ZH"
- note added: "JST-ZH Connectors"
- note added: "MOTOR DRIVERS"
- note added: "Overcharge Protection at 4.3V Overcharge timeout td = C19 * 9.0s/uF = 0.9 seconds Discharge Protection at 2.5V CHG_EN goes HIGH to disable charger"
- note added: "Prototyping Power Rails"
- note added: "SD-101D"
- note added: "Servo Connectors & Power Control"
- note added: "Servo Pulldowns"
- note added: "Strawson Design Robotics Cape Rev. D"
- note added: "eQEP Encoder Plugs JST SH"
- note added: "green"
- note added: "red"
- moved on the sheet: R112
