File: Eagle/BeagleBone_Blue.brd (EAGLE design)
At the start: 86.4 x 54.6 mm, 125 parts, among them M1 JST_ZH_2, M2 JST_ZH_2, M3 JST_ZH_2, M4 JST_ZH_2, Q3 MOSFET-N

Commit message: Shuffle components on the board
Parts:
- moved DSM2 34.0 mm to (12.6, 23.9)
- moved UART5 26.8 mm to (47.1, 13.8)
- moved UART1 26.1 mm to (47.1, 23.4)
- moved GPS 25.3 mm to (26.2, 19.7)
- moved SPI1.2 25.2 mm to (31.0, 19.8)
- moved ADC 25.1 mm to (40.4, 19.4)
- moved SPI1.1 24.8 mm to (35.8, 19.6)
- moved R13 23.1 mm to (22.6, 29.2)
- moved PWR 22.8 mm to (17.7, 23.4)
- moved I2C1 22.5 mm to (22.5, 23.1)
- moved C16 21.5 mm to (18.3, 27.9)
- moved R12 21.2 mm to (21.0, 29.2)
- moved U$5 12.9 mm to (57.8, 13.3)
- flipped BMP to the bottom

Commit message: Initial USB connector placement
Parts:
- added C34: (no value), BeagleBone_Blue:AVE107M06D16T-F
- added CLIENT: (no value), BeagleBone_Blue:UX60SC-MB-5ST(80)
- added HOST: (no value), BeagleBone_Blue:87520-0010BLF
- moved SIP 13.0 mm to (45.3, 27.9)
- moved BMP 11.4 mm to (55.4, 5.21)
Changed lines of the file:
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@@
 <attribute name="NAME" x="59.2455" y="25.781" size="0.508" layer="25" rot="R90"/>
 </element>
-<element name="BMP" library="SparkFun-Sensors" package="BMP180" value="BMP180" x="54.864" y="16.637" smashed="yes" rot="MR0">
-<attribute name="NAME" x="56.039" y="17.113" size="0.508" layer="26" rot="MR270"/>
+<element name="BMP" library="SparkFun-Sensors" package="BMP180" value="BMP180" x="55.372" y="5.207" smashed="yes" rot="MR0">
+<attribute name="NAME" x="56.547" y="5.683" size="0.508" layer="26" rot="MR270"/>
 </element>
 <element name="C13" library="Strawson_Eagle_Lib" package="0402-CAP" value="0.1uF" x="58.42" y="19.685" smashed="yes" rot="R270">
@@
 </element>
 <element name="U$7" library="Strawson_Eagle_Lib" package="BEAGLEBONE_BLUE_NO_HOLES" value="" x="0" y="54.61" rot="R270"/>
-<element name="SIP" library="BeagleBone_Blue" package="OSD3358" value="" x="32.639" y="25.146" rot="MR0"/>
+<element name="SIP" library="BeagleBone_Blue" package="OSD3358" value="" x="45.339" y="27.94" rot="MR0"/>
 <element name="BOOT" library="SparkFun-Electromechanical" package="TACTILE-SWITCH-1101NE" value="SWITCH-MOMENTARY-2-SMD-1101NE" x="5.207" y="43.688" smashed="yes">
 <attribute name="NAME" x="15.621" y="44.323" size="1.524" layer="25" ratio="10" rot="R180"/>
 </element>
 <element name="P10" library="SCHA5B0200" package="SCHA5B0200" value="" x="80.772" y="-0.762" rot="MR0"/>
+<element name="C34" library="BeagleBone_Blue" package="AVE107M06D16T-F" value="" x="68.072" y="6.604"/>
+<element name="CLIENT" library="BeagleBone_Blue" package="UX60SC-MB-5ST(80)" value="" x="45.847" y="19.431" rot="R90"/>
+<element name="HOST" library="BeagleBone_Blue" package="87520-0010BLF" value="" x="36.322" y="7.493"/>
 </elements>
 <signals>
@@
 <wire x1="55.614" y1="21.368" x2="55.614" y2="20.8668" width="0.254" layer="1"/>
 <wire x1="55.614" y1="20.8668" x2="55.245" y2="20.3708" width="0.254" layer="1"/>
-<wire x1="54.864" y1="15.187" x2="55.245" y2="20.3708" width="0" layer="19" extent="1-1"/>
+<wire x1="55.372" y1="3.757" x2="55.245" y2="20.3708" width="0" layer="19" extent="1-1"/>
 </signal>
 <signal name="I2C2_SDA">
@@
 <wire x1="56.114" y1="21.368" x2="56.114" y2="20.3908" width="0.254" layer="1"/>
 <wire x1="56.114" y1="20.3908" x2="56.134" y2="20.3708" width="0.254" layer="1"/>
-<wire x1="53.364" y1="15.187" x2="56.134" y2="20.3708" width="0" layer="19" extent="1-1"/>
+<wire x1="53.872" y1="3.757" x2="56.134" y2="20.3708" width="0" layer="19" extent="1-1"/>
 </signal>
 <signal name="PWM_2B">
@@
 <wire x1="56.134" y1="19.2532" x2="56.864" y2="23.118" width="0" layer="19" extent="1-1"/>
 <wire x1="58.42" y1="20.2438" x2="56.134" y2="19.2532" width="0" layer="19" extent="1-1"/>
-<wire x1="54.864" y1="18.087" x2="56.261" y2="17.1958" width="0" layer="19" extent="1-1"/>
-<wire x1="56.364" y1="18.087" x2="54.864" y2="18.087" width="0" layer="19" extent="1-1"/>
+<wire x1="55.372" y1="6.657" x2="56.261" y2="17.1958" width="0" layer="19" extent="1-1"/>
+<wire x1="56.872" y1="6.657" x2="55.372" y2="6.657" width="0" layer="19" extent="1-1"/>
 <wire x1="64.389" y1="18.4658" x2="56.261" y2="17.1958" width="0" layer="19" extent="1-1"/>
-<wire x1="35.814" y1="23.558" x2="56.364" y2="18.087" width="0" layer="19" extent="1-1"/>
+<wire x1="35.814" y1="23.558" x2="56.872" y2="6.657" width="0" layer="19" extent="1-1"/>
 <wire x1="30.988" y1="23.812" x2="35.814" y2="23.558" width="0" layer="19" extent="1-1"/>
 <wire x1="12.573" y1="23.876" x2="30.988" y2="23.812" width="0" layer="19" extent="1-1"/>
@@
 <wire x1="26.162" y1="19.685" x2="12.573" y2="22.3774" width="0" layer="19" extent="1-1"/>
 <wire x1="58.42" y1="19.1262" x2="56.864" y2="22.118" width="0" layer="19" extent="1-1"/>
-<wire x1="53.364" y1="16.637" x2="58.42" y2="19.1262" width="0" layer="19" extent="1-1"/>
+<wire x1="53.872" y1="5.207" x2="58.42" y2="19.1262" width="0" layer="19" extent="1-1"/>
 <wire x1="63.119" y1="29.197" x2="58.42" y2="26.9748" width="0" layer="19" extent="1-1"/>
 <wire x1="61.087" y1="32.9565" x2="63.119" y2="29.197" width="0" layer="19" extent="1-1"/>
