File: EAGLE_SIP/BeagleBone_Blue.brd (EAGLE design)
At the start: 86.4 x 54.6 mm, 279 parts, among them M1 JST_ZH_2, M2 JST_ZH_2, M3 JST_ZH_2, M4 JST_ZH_2, P10 SCHA5B0200, Q3 MOSFET-N, U1 TPD4S012_DRY_6, U4 TPD4S012_DRY_6, U5 24LC_32AT-I/OT, U6 SN74LVC1G07_DCK_5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

Commit message: Rough place some parts
Parts:
- moved C9 33.0 mm to (20.3, -24.8), turned to 90 degrees
- moved C4 14.2 mm to (38.7, -7.94)
- moved R19 2.71 mm to (43.9, -8.57)

Commit message: Rough place some parts
Parts:
- moved C14 40.2 mm to (36.8, -7.94)
- moved C4 0.63 mm to (39.4, -7.94)
Changed lines of the file:
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@@
 <element name="C12" library="SparkFun-Capacitors" package="0805" value="10uF 25V" x="33.147" y="-4.445" rot="R90"/>
 <element name="C13" library="Strawson_Eagle_Lib" package="0402-CAP" value="0.1uF" x="11.811" y="-22.479" rot="R90"/>
-<element name="C14" library="Strawson_Eagle_Lib" package="0402-CAP" value="0.1uF" x="-0.889" y="5.969"/>
+<element name="C14" library="Strawson_Eagle_Lib" package="0402-CAP" value="0.1uF" x="36.83" y="-7.9375"/>
 <element name="C15" library="Strawson_Eagle_Lib" package="0402-CAP" value="0.1uF" x="-3.429" y="5.969"/>
 <element name="C16" library="SparkFun-Capacitors" package="0805" value="10uF 25V" x="24.765" y="-18.288"/>
@@
 <element name="C38" library="Strawson_Eagle_Lib" package="0805" value="10UF,10V" x="53.0225" y="-50.165" rot="MR90"/>
 <element name="C39" library="Strawson_Eagle_Lib" package="0402-CAP" value="0.1UF,6.3V" x="39.0525" y="-43.4975" rot="R90"/>
-<element name="C4" library="Strawson_Eagle_Lib" package="0402-CAP" value="1uF" x="38.735" y="-7.9375"/>
+<element name="C4" library="Strawson_Eagle_Lib" package="0402-CAP" value="1uF" x="39.37" y="-7.9375"/>
 <element name="C40" library="Strawson_Eagle_Lib" package="0402-CAP" value="0.1UF,6.3V" x="38.735" y="-52.07" rot="R90"/>
 <element name="C41" library="Strawson_Eagle_Lib" package="0402-CAP" value="0.1UF,6.3V" x="52.705" y="-44.1325" rot="MR90"/>
@@
 <wire x1="46.5582" y1="-13.335" x2="43.887" y2="-12.7" width="0" layer="19" extent="1-1"/>
 <wire x1="41.402" y1="-8.9662" x2="43.887" y2="-12.7" width="0" layer="19" extent="1-1"/>
-<wire x1="38.1762" y1="-7.9375" x2="41.402" y2="-8.9662" width="0" layer="19" extent="1-1"/>
-<wire x1="36.2077" y1="-5.969" x2="38.1762" y2="-7.9375" width="0" layer="19" extent="1-1"/>
+<wire x1="38.8112" y1="-7.9375" x2="41.402" y2="-8.9662" width="0" layer="19" extent="1-1"/>
+<wire x1="36.2077" y1="-5.969" x2="38.8112" y2="-7.9375" width="0" layer="19" extent="1-1"/>
 <wire x1="39.1033" y1="-3.937" x2="36.2077" y2="-5.969" width="0" layer="19" extent="1-1"/>
 <wire x1="38.4285" y1="-1.3335" x2="39.1033" y2="-3.937" width="0" layer="19" extent="1-1"/>
@@
 <wire x1="16.475" y1="-23.546" x2="15.875" y2="-25.146" width="0" layer="19" extent="1-1"/>
 <wire x1="17.475" y1="-24.146" x2="16.475" y2="-23.546" width="0" layer="19" extent="1-1"/>
-<wire x1="12.446" y1="-30.353" x2="12.7" y2="-26.9748" width="0" layer="19" extent="1-1"/>
 <wire x1="20.32" y1="-25.3238" x2="17.475" y2="-24.146" width="0" layer="19" extent="1-1"/>
 <wire x1="21.1582" y1="-27.94" x2="20.32" y2="-25.3238" width="0" layer="19" extent="1-1"/>
+<wire x1="12.446" y1="-30.353" x2="12.7" y2="-26.9748" width="0" layer="19" extent="1-1"/>
 <wire x1="56.261" y1="-7.487" x2="54.2798" y2="-14.732" width="0" layer="19" extent="1-1"/>
 <wire x1="57.531" y1="-7.487" x2="56.261" y2="-7.487" width="0" layer="19" extent="1-1"/>
@@
 <contactref element="CHGIC" pad="15"/>
 <contactref element="C14" pad="1"/>
-<wire x1="-1.4478" y1="5.969" x2="36.2077" y2="-5.461" width="0" layer="19" extent="1-1"/>
+<wire x1="36.2712" y1="-7.9375" x2="36.2077" y2="-5.461" width="0" layer="19" extent="1-1"/>
 </signal>
 <signal name="N$55">
@@
 <contactref element="L2" pad="1"/>
 <wire x1="37.1475" y1="-6.0452" x2="44.625" y2="-5.858" width="0" layer="19" extent="1-1"/>
-<wire x1="-0.3302" y1="5.969" x2="37.1475" y2="-6.0452" width="0" layer="19" extent="1-1"/>
+<wire x1="37.3888" y1="-7.9375" x2="37.1475" y2="-6.0452" width="0" layer="19" extent="1-1"/>
 </signal>
 <signal name="N$67">
@@
 <contactref element="CHGIC" pad="5"/>
 <wire x1="39.1033" y1="-5.461" x2="38.1635" y2="-6.0452" width="0" layer="19" extent="1-1"/>
-<wire x1="39.2938" y1="-7.9375" x2="38.1635" y2="-6.0452" width="0" layer="19" extent="1-1"/>
-<wire x1="37.5158" y1="-13.97" x2="39.2938" y2="-7.9375" width="0" layer="19" extent="1-1"/>
+<wire x1="39.9288" y1="-7.9375" x2="38.1635" y2="-6.0452" width="0" layer="19" extent="1-1"/>
+<wire x1="37.5158" y1="-13.97" x2="39.9288" y2="-7.9375" width="0" layer="19" extent="1-1"/>
 </signal>
 <signal name="N$71">

Commit message: Rough place some parts
Parts:
- moved C15 54.8 mm to (49.5, -7.94)
Changed lines of the file:
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@@
 <element name="C13" library="Strawson_Eagle_Lib" package="0402-CAP" value="0.1uF" x="11.811" y="-22.479" rot="R90"/>
 <element name="C14" library="Strawson_Eagle_Lib" package="0402-CAP" value="0.1uF" x="36.83" y="-7.9375"/>
-<element name="C15" library="Strawson_Eagle_Lib" package="0402-CAP" value="0.1uF" x="-3.429" y="5.969"/>
+<element name="C15" library="Strawson_Eagle_Lib" package="0402-CAP" value="0.1uF" x="49.53" y="-7.9375"/>
 <element name="C16" library="SparkFun-Capacitors" package="0805" value="10uF 25V" x="24.765" y="-18.288"/>
 <element name="C17" library="Strawson_Eagle_Lib" package="0402-CAP" value="0.1uF" x="49.911" y="-4.191"/>
@@
 <wire x1="57.531" y1="-13.087" x2="56.261" y2="-13.087" width="0" layer="19" extent="1-1"/>
 <wire x1="58.801" y1="-13.087" x2="57.531" y2="-13.087" width="0" layer="19" extent="1-1"/>
-<wire x1="-3.9878" y1="5.969" x2="50.4698" y2="-1.397" width="0" layer="19" extent="1-1"/>
-<wire x1="-9.0678" y1="5.969" x2="-3.9878" y2="5.969" width="0" layer="19" extent="1-1"/>
+<wire x1="48.9712" y1="-7.9375" x2="50.4698" y2="-1.397" width="0" layer="19" extent="1-1"/>
+<wire x1="-9.0678" y1="5.969" x2="48.9712" y2="-7.9375" width="0" layer="19" extent="1-1"/>
 </signal>
 <signal name="N$8">
@@
 <contactref element="R44" pad="2"/>
 <wire x1="51.6382" y1="-8.382" x2="61.087" y2="-8.1788" width="0" layer="19" extent="1-16"/>
-<wire x1="-2.8702" y1="5.969" x2="51.6382" y2="-8.382" width="0" layer="19" extent="1-1"/>
+<wire x1="50.0888" y1="-7.9375" x2="51.6382" y2="-8.382" width="0" layer="19" extent="1-1"/>
 </signal>
 <signal name="DO">

Commit message: Rough place some parts
Parts:
- moved C18 62.0 mm to (53.0, -1.27), turned to 180 degrees
- moved BAL 0.64 mm to (53.5, -4.06)
Changed lines of the file:
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@@
 <attribute name="NAME" x="58.801" y="-48.7045" size="1.016" layer="25" rot="R180"/>
 </element>
-<element name="BAL" library="Strawson_Eagle_Lib" package="8-SON_3X3MM" value="BQ29209" x="53.467" y="-3.429"/>
+<element name="BAL" library="Strawson_Eagle_Lib" package="8-SON_3X3MM" value="BQ29209" x="53.467" y="-4.064"/>
 <element name="BMP" library="SparkFun-Sensors" package="BMP180" value="BMP180" x="66.802" y="-29.845" rot="MR0"/>
 <element name="BOOT" library="SparkFun-Electromechanical" package="TACTILE-SWITCH-1101NE" value="SWITCH-MOMENTARY-2SMD-1101NE" x="4.699" y="-36.449" smashed="yes">
@@
 <element name="C16" library="SparkFun-Capacitors" package="0805" value="10uF 25V" x="24.765" y="-18.288"/>
 <element name="C17" library="Strawson_Eagle_Lib" package="0402-CAP" value="0.1uF" x="49.911" y="-4.191"/>
-<element name="C18" library="Strawson_Eagle_Lib" package="0402-CAP" value="0.1uF" x="-8.509" y="5.969"/>
+<element name="C18" library="Strawson_Eagle_Lib" package="0402-CAP" value="0.1uF" x="53.0225" y="-1.27" rot="R180"/>
 <element name="C19" library="Strawson_Eagle_Lib" package="0402-CAP" value="0.1uF" x="86.741" y="9.779"/>
 <element name="C2" library="Strawson_Eagle_Lib" package="0402-CAP" value="0.1uF" x="81.5975" y="-26.67"/>
@@
 <contactref element="R30" pad="2"/>
 <contactref element="BAL" pad="2"/>
-<wire x1="49.3522" y1="-4.191" x2="53.1368" y2="-4.9022" width="0" layer="19" extent="1-1"/>
+<wire x1="53.1368" y1="-5.5372" x2="52.4637" y2="-1.27" width="0" layer="19" extent="1-1"/>
+<wire x1="49.3522" y1="-4.191" x2="53.1368" y2="-5.5372" width="0" layer="19" extent="1-1"/>
 <wire x1="45.212" y1="-10.2362" x2="49.3522" y2="-4.191" width="0" layer="19" extent="1-1"/>
-<wire x1="-7.9502" y1="5.969" x2="45.212" y2="-10.2362" width="0" layer="19" extent="1-1"/>
 </signal>
 <signal name="BATT_MINUS">
@@
 <contactref element="PROT" pad="2"/>
 <wire x1="58.547" y1="-3.81" x2="87.2998" y2="9.779" width="0" layer="19" extent="1-1"/>
-<wire x1="54.4322" y1="-1.9558" x2="58.547" y2="-3.81" width="0" layer="19" extent="1-1"/>
-<wire x1="53.7972" y1="-1.9558" x2="54.4322" y2="-1.9558" width="0" layer="19" extent="1-1"/>
-<wire x1="50.4698" y1="-1.397" x2="53.7972" y2="-1.9558" width="0" layer="19" extent="1-1"/>
+<wire x1="54.4322" y1="-2.5908" x2="58.547" y2="-3.81" width="0" layer="19" extent="1-1"/>
+<wire x1="53.7972" y1="-2.5908" x2="54.4322" y2="-2.5908" width="0" layer="19" extent="1-1"/>
+<wire x1="53.5813" y1="-1.27" x2="53.7972" y2="-2.5908" width="0" layer="19" extent="1-1"/>
+<wire x1="50.4698" y1="-1.397" x2="53.5813" y2="-1.27" width="0" layer="19" extent="1-1"/>
 <wire x1="54.0258" y1="-8.382" x2="58.547" y2="-3.81" width="0" layer="19" extent="1-1"/>
 <wire x1="51.6382" y1="-9.3218" x2="54.0258" y2="-8.382" width="0" layer="19" extent="1-1"/>
+<wire x1="48.9712" y1="-7.9375" x2="51.6382" y2="-9.3218" width="0" layer="19" extent="1-1"/>
 <wire x1="56.261" y1="-13.087" x2="54.0258" y2="-8.382" width="0" layer="19" extent="1-1"/>
 <wire x1="57.531" y1="-13.087" x2="56.261" y2="-13.087" width="0" layer="19" extent="1-1"/>
 <wire x1="58.801" y1="-13.087" x2="57.531" y2="-13.087" width="0" layer="19" extent="1-1"/>
-<wire x1="48.9712" y1="-7.9375" x2="50.4698" y2="-1.397" width="0" layer="19" extent="1-1"/>
-<wire x1="-9.0678" y1="5.969" x2="48.9712" y2="-7.9375" width="0" layer="19" extent="1-1"/>
 </signal>
 <signal name="N$8">
@@
 <contactref element="C17" pad="2"/>
 <contactref element="BAL" pad="1"/>
-<wire x1="50.4698" y1="-4.191" x2="52.5018" y2="-4.9022" width="0" layer="19" extent="1-1"/>
+<wire x1="50.4698" y1="-4.191" x2="52.5018" y2="-5.5372" width="0" layer="19" extent="1-1"/>
 <wire x1="43.8658" y1="-10.16" x2="50.4698" y2="-4.191" width="0" layer="19" extent="1-1"/>
 </signal>
@@
 <contactref element="BAL" pad="7"/>
 <contactref element="C1" pad="1"/>
-<wire x1="50.4698" y1="-2.794" x2="53.1368" y2="-1.9558" width="0" layer="19" extent="1-1"/>
+<wire x1="50.4698" y1="-2.794" x2="53.1368" y2="-2.5908" width="0" layer="19" extent="1-1"/>
 <wire x1="49.3522" y1="-1.397" x2="50.4698" y2="-2.794" width="0" layer="19" extent="1-1"/>
 </signal>
@@
 <contactref element="BAL" pad="4"/>
 <contactref element="C19" pad="1"/>
-<wire x1="54.4322" y1="-4.9022" x2="86.1822" y2="9.779" width="0" layer="19" extent="1-1"/>
+<wire x1="54.4322" y1="-5.5372" x2="86.1822" y2="9.779" width="0" layer="19" extent="1-1"/>
 </signal>
 <signal name="N$50">
 <contactref element="R27" pad="2"/>
 <contactref element="BAL" pad="3"/>
-<wire x1="46.5582" y1="-10.16" x2="53.7972" y2="-4.9022" width="0" layer="19" extent="1-1"/>
+<wire x1="46.5582" y1="-10.16" x2="53.7972" y2="-5.5372" width="0" layer="19" extent="1-1"/>
 </signal>
 <signal name="CO">
 <contactref element="BAL" pad="8"/>
 <contactref element="R7" pad="1"/>
-<wire x1="40.2082" y1="-11.43" x2="52.5018" y2="-1.9558" width="0" layer="19" extent="1-1"/>
+<wire x1="40.2082" y1="-11.43" x2="52.5018" y2="-2.5908" width="0" layer="19" extent="1-1"/>
 </signal>
 <signal name="N$11">

Commit message: Rough place some parts
Parts:
- moved C21 40.6 mm to (65.1, -26.0), turned to 270 degrees
- moved C22 38.7 mm to (64.1, -24.8), flipped to the bottom, turned to 180 degrees
- moved C19 35.4 mm to (55.2, -6.35), flipped to the bottom, turned to 180 degrees
Changed lines of the file:
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@@
 <element name="C17" library="Strawson_Eagle_Lib" package="0402-CAP" value="0.1uF" x="49.911" y="-4.191"/>
 <element name="C18" library="Strawson_Eagle_Lib" package="0402-CAP" value="0.1uF" x="53.0225" y="-1.27" rot="R180"/>
-<element name="C19" library="Strawson_Eagle_Lib" package="0402-CAP" value="0.1uF" x="86.741" y="9.779"/>
+<element name="C19" library="Strawson_Eagle_Lib" package="0402-CAP" value="0.1uF" x="55.245" y="-6.35" rot="MR180"/>
 <element name="C2" library="Strawson_Eagle_Lib" package="0402-CAP" value="0.1uF" x="81.5975" y="-26.67"/>
 <element name="C20" library="SparkFun-Capacitors" package="0805" value="10uF 25V" x="60.325" y="-23.1775"/>
-<element name="C21" library="Strawson_Eagle_Lib" package="0402-CAP" value="2.2nF 50V" x="84.201" y="9.779"/>
-<element name="C22" library="Strawson_Eagle_Lib" package="0402-CAP" value="0.1uF" x="81.661" y="9.779"/>
+<element name="C21" library="Strawson_Eagle_Lib" package="0402-CAP" value="2.2nF 50V" x="65.0875" y="-26.035" rot="R270"/>
+<element name="C22" library="Strawson_Eagle_Lib" package="0402-CAP" value="0.1uF" x="64.135" y="-24.765" rot="MR180"/>
 <element name="C23" library="SparkFun-Capacitors" package="0805" value="10uF 25V" x="63.8175" y="-23.1775"/>
 <element name="C24" library="Strawson_Eagle_Lib" package="0402-CAP" value="0.1uF" x="79.121" y="9.779"/>
@@
 <contactref element="R17" pad="2"/>
 <contactref element="R9" pad="2"/>
-<wire x1="78.5622" y1="9.779" x2="83.6422" y2="9.779" width="0" layer="19" extent="1-1"/>
+<wire x1="78.5622" y1="9.779" x2="65.0875" y2="-25.4762" width="0" layer="19" extent="1-1"/>
 <wire x1="77.1398" y1="9.779" x2="78.5622" y2="9.779" width="0" layer="19" extent="1-1"/>
 <wire x1="74.5998" y1="9.779" x2="77.1398" y2="9.779" width="0" layer="19" extent="1-1"/>
@@
 <contactref element="C15" pad="1"/>
 <contactref element="PROT" pad="2"/>
-<wire x1="58.547" y1="-3.81" x2="87.2998" y2="9.779" width="0" layer="19" extent="1-1"/>
+<wire x1="58.547" y1="-3.81" x2="55.8038" y2="-6.35" width="0" layer="19" extent="1-1"/>
 <wire x1="54.4322" y1="-2.5908" x2="58.547" y2="-3.81" width="0" layer="19" extent="1-1"/>
 <wire x1="53.7972" y1="-2.5908" x2="54.4322" y2="-2.5908" width="0" layer="19" extent="1-1"/>
@@
 <contactref element="BAL" pad="4"/>
 <contactref element="C19" pad="1"/>
-<wire x1="54.4322" y1="-5.5372" x2="86.1822" y2="9.779" width="0" layer="19" extent="1-1"/>
+<wire x1="54.4322" y1="-5.5372" x2="54.6862" y2="-6.35" width="0" layer="19" extent="1-1"/>
 </signal>
 <signal name="N$50">
@@
 <contactref element="6V_REG" pad="7"/>
 <contactref element="C21" pad="2"/>
-<wire x1="63.252" y1="-26.543" x2="84.7598" y2="9.779" width="0" layer="19" extent="1-1"/>
+<wire x1="63.252" y1="-26.543" x2="65.0875" y2="-26.5938" width="0" layer="19" extent="1-1"/>
 </signal>
 <signal name="SERVO_EN">
@@
 <contactref element="6V_REG" pad="2"/>
 <contactref element="C22" pad="1"/>
-<wire x1="57.652" y1="-26.543" x2="81.1022" y2="9.779" width="0" layer="19" extent="1-1"/>
+<wire x1="57.652" y1="-26.543" x2="63.5762" y2="-24.765" width="0" layer="19" extent="1-1"/>
 </signal>
 <signal name="N$60">
@@
 <contactref element="D9" pad="C"/>
 <contactref element="L3" pad="1"/>
-<wire x1="70.739" y1="-24.892" x2="82.2198" y2="9.779" width="0" layer="19" extent="1-1"/>
+<wire x1="70.739" y1="-24.892" x2="64.6938" y2="-24.765" width="0" layer="19" extent="1-1"/>
 <wire x1="73.4695" y1="-33.909" x2="70.739" y2="-24.892" width="0" layer="19" extent="1-1"/>
 <wire x1="57.652" y1="-25.273" x2="70.739" y2="-24.892" width="0" layer="19" extent="1-1"/>

Commit message: Rough place some parts
Parts:
- moved C27 43.9 mm to (52.8, -27.1)
- moved C24 34.5 mm to (64.1, -21.3), turned to 180 degrees

Commit message: Rough place some parts
Parts:
- moved C28 57.8 mm to (25.1, -21.0)

Commit message: Rough place some parts
Parts:
- moved C36 58.7 mm to (39.1, -46.4), turned to 90 degrees
Changed lines of the file:
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@@
 <attribute name="NAME" x="74.803" y="-46.5455" size="0.4064" layer="25"/>
 </element>
-<element name="C36" library="Strawson_Eagle_Lib" package="0402-CAP" value="2.2UF,6.3V" x="56.261" y="9.779"/>
+<element name="C36" library="Strawson_Eagle_Lib" package="0402-CAP" value="2.2UF,6.3V" x="39.0525" y="-46.355" rot="R90"/>
 <element name="C37" library="Strawson_Eagle_Lib" package="0402-CAP" value="0.1UF,6.3V" x="52.3875" y="-53.6575"/>
 <element name="C38" library="Strawson_Eagle_Lib" package="0805" value="10UF,10V" x="53.0225" y="-50.165" rot="MR90"/>
@@
 <wire x1="24.003" y1="-68.7578" x2="25.908" y2="-67.6402" width="0" layer="19" extent="1-1"/>
 <wire x1="49.1998" y1="17.399" x2="36.4998" y2="9.779" width="0" layer="19" extent="1-1"/>
-<wire x1="55.7022" y1="9.779" x2="49.1998" y2="17.399" width="0" layer="19" extent="1-1"/>
+<wire x1="39.0525" y1="-46.9138" x2="49.1998" y2="17.399" width="0" layer="19" extent="1-1"/>
 </signal>
 <signal name="N$6">
@@
 <contactref element="C36" pad="2"/>
 <contactref element="U8" pad="C2"/>
-<wire x1="42.327" y1="-45.1925" x2="56.8198" y2="9.779" width="0" layer="19" extent="1-16"/>
+<wire x1="42.327" y1="-45.1925" x2="39.0525" y2="-45.7962" width="0" layer="19" extent="1-16"/>
 </signal>
 <signal name="N$111">
