File: EAGLE_SIP/BeagleBone_Blue.brd (EAGLE design)
At the start: 86.4 x 54.6 mm, 263 parts, among them M1 JST_ZH_2, M2 JST_ZH_2, M3 JST_ZH_2, M4 JST_ZH_2, P10 SCHA5B0200, Q3 MOSFET-N, U1 TPD4S012_DRY_6, U4 TPD4S012_DRY_6, U5 24LC_32AT-I/OT, U6 SN74LVC1G07_DCK_5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

Commit message: Delete some test points I know I will not use
Parts:
- removed TP2: TPSQB1,27, testpad:B1,27
- moved TP1 1.35 mm to (55.7, -42.9), turned to 180 degrees
Connections:
- removed net N$5: SIP.Y2, SIP.Y3, TP2.TP
- new net VIN_BAT_0: SIP.Y2
- new net VIN_BAT_1: SIP.Y3
